File: kicad_SchalterFahrakku/Schalter_Fahrakku.sch (KiCad schematic (older format))
At the start: 15 parts, among them P1 V+_IN, P2 V-_IN, P3 V+_OUT, P4 V-_OUT, Q1 IRLML6344, Q2 IPD90P03

Commit message: - Neue anschlüsse in Schalterplatine eingefügt
Parts:
- removed P1: V+_IN, Wire_Pads:SolderWirePad_single_SMD_5x10mm, symbol CONN_01X01
- removed P2: V-_IN, Wire_Pads:SolderWirePad_single_SMD_5x10mm, symbol CONN_01X01
- removed P3: V+_OUT, Wire_Pads:SolderWirePad_single_SMD_5x10mm, symbol CONN_01X01
- removed P4: V-_OUT, Wire_Pads:SolderWirePad_single_SMD_5x10mm, symbol CONN_01X01
- added P1: V_IN, Custom:AKL_320-02, symbol CONN_01X02
- added P2: V_OUT, Custom:AKL_320-02, symbol CONN_01X02
- PD1, PD2, PD3, PD4: footprint Mounting_Holes:MountingHole_3.2mm_M3 -> Custom:MountingHole_3.3mm_M3
Connections:
- wire segments 18 -> 25
Changed lines of the file:
@@
 $EndComp
 $Comp
-L GND #PWR3
+L GND #PWR01
 U 1 1 5783BA47
 P 4450 4350
-F 0 "#PWR3" H 4450 4100 50  0001 C CNN
+F 0 "#PWR01" H 4450 4100 50  0001 C CNN
 F 1 "GND" H 4450 4200 50  0000 C CNN
 F 2 "" H 4450 4350 50  0000 C CNN
@@
 $EndComp
 $Comp
-L GND #PWR4
+L GND #PWR02
 U 1 1 5783BA63
 P 4850 4150
-F 0 "#PWR4" H 4850 3900 50  0001 C CNN
+F 0 "#PWR02" H 4850 3900 50  0001 C CNN
 F 1 "GND" H 4850 4000 50  0000 C CNN
 F 2 "" H 4850 4150 50  0000 C CNN
@@
 $EndComp
 $Comp
-L GND #PWR2
+L GND #PWR03
 U 1 1 5783C373
-P 4000 3275
-F 0 "#PWR2" H 4000 3025 50  0001 C CNN
-F 1 "GND" H 4000 3125 50  0000 C CNN
-F 2 "" H 4000 3275 50  0000 C CNN
-F 3 "" H 4000 3275 50  0000 C CNN
-	1    4000 3275
-	1    0    0    -1
-$EndComp
-$Comp
-L GND #PWR1
+P 4000 3325
+F 0 "#PWR03" H 4000 3075 50  0001 C CNN
+F 1 "GND" H 4000 3175 50  0000 C CNN
+F 2 "" H 4000 3325 50  0000 C CNN
+F 3 "" H 4000 3325 50  0000 C CNN
+	1    4000 3325
+	1    0    0    -1
+$EndComp
+$Comp
+L GND #PWR04
 U 1 1 5783C4FA
 P 3950 3800
-F 0 "#PWR1" H 3950 3550 50  0001 C CNN
+F 0 "#PWR04" H 3950 3550 50  0001 C CNN
 F 1 "GND" H 3950 3650 50  0000 C CNN
 F 2 "" H 3950 3800 50  0000 C CNN
@@
 $EndComp
 $Comp
-L GND #PWR5
+L GND #PWR05
 U 1 1 5783C5FB
 P 5750 3350
-F 0 "#PWR5" H 5750 3100 50  0001 C CNN
+F 0 "#PWR05" H 5750 3100 50  0001 C CNN
 F 1 "GND" H 5750 3200 50  0000 C CNN
 F 2 "" H 5750 3350 50  0000 C CNN
@@
 Connection ~ 4450 2900
 Wire Wire Line
-	4000 2900 5150 2900
-Wire Wire Line
-	5750 2900 5550 2900
+	3950 2900 5150 2900
+Wire Wire Line
+	5550 2900 6025 2900
 Wire Wire Line
 	5750 3350 5750 3350
@@
 Connection ~ 4175 3900
 $Comp
-L CONN_01X01 P1
-U 1 1 57ADC701
-P 3800 2900
-F 0 "P1" H 3800 3000 50  0000 C CNN
-F 1 "V+_IN" V 3900 2900 50  0000 C CNN
-F 2 "Wire_Pads:SolderWirePad_single_SMD_5x10mm" H 3800 2900 50  0001 C CNN
-F 3 "" H 3800 2900 50  0000 C CNN
-F 4 "Pad" H 3800 2900 60  0001 C CNN "Package"
-	1    3800 2900
-	-1   0    0    1
-$EndComp
-$Comp
-L CONN_01X01 P2
-U 1 1 57ADC760
-P 3800 3275
-F 0 "P2" H 3800 3375 50  0000 C CNN
-F 1 "V-_IN" V 3900 3275 50  0000 C CNN
-F 2 "Wire_Pads:SolderWirePad_single_SMD_5x10mm" H 3800 3275 50  0001 C CNN
-F 3 "" H 3800 3275 50  0000 C CNN
-F 4 "Pad" H 3800 3275 60  0001 C CNN "Package"
-	1    3800 3275
-	-1   0    0    1
-$EndComp
-$Comp
-L CONN_01X01 P3
-U 1 1 57ADC7D4
-P 5950 2900
-F 0 "P3" H 5950 3000 50  0000 C CNN
-F 1 "V+_OUT" V 6050 2900 50  0000 C CNN
-F 2 "Wire_Pads:SolderWirePad_single_SMD_5x10mm" H 5950 2900 50  0001 C CNN
-F 3 "" H 5950 2900 50  0000 C CNN
-F 4 "Pad" H 5950 2900 60  0001 C CNN "Package"
-	1    5950 2900
-	1    0    0    1
-$EndComp
-$Comp
-L CONN_01X01 P4
-U 1 1 57ADC84B
-P 5950 3350
-F 0 "P4" H 5950 3450 50  0000 C CNN
-F 1 "V-_OUT" V 6050 3350 50  0000 C CNN
-F 2 "Wire_Pads:SolderWirePad_single_SMD_5x10mm" H 5950 3350 50  0001 C CNN
-F 3 "" H 5950 3350 50  0000 C CNN
-F 4 "Pad" H 5950 3350 60  0001 C CNN "Package"
-	1    5950 3350
-	1    0    0    1
-$EndComp
-$Comp
 L R_Small R2
 U 1 1 57ADCAFA
@@
 Connection ~ 5075 2900
 $Comp
-L PWR_FLAG #FLG1
+L PWR_FLAG #FLG06
 U 1 1 57ADD4B4
 P 4000 2900
-F 0 "#FLG1" H 4000 2995 50  0001 C CNN
+F 0 "#FLG06" H 4000 2995 50  0001 C CNN
 F 1 "PWR_FLAG" H 4000 3080 50  0000 C CNN
 F 2 "" H 4000 2900 50  0000 C CNN
@@
 $EndComp
 $Comp
-L PWR_FLAG #FLG2
+L PWR_FLAG #FLG07
 U 1 1 57ADD513
-P 4000 3275
-F 0 "#FLG2" H 4000 3370 50  0001 C CNN
-F 1 "PWR_FLAG" H 4000 3455 50  0000 C CNN
-F 2 "" H 4000 3275 50  0000 C CNN
-F 3 "" H 4000 3275 50  0000 C CNN
-	1    4000 3275
-	1    0    0    -1
-$EndComp
-$Comp
-L PWR_FLAG #FLG3
+P 4200 3250
+F 0 "#FLG07" H 4200 3345 50  0001 C CNN
+F 1 "PWR_FLAG" H 4200 3430 50  0000 C CNN
+F 2 "" H 4200 3250 50  0000 C CNN
+F 3 "" H 4200 3250 50  0000 C CNN
+	1    4200 3250
+	1    0    0    -1
+$EndComp
+$Comp
+L PWR_FLAG #FLG08
 U 1 1 57ADD53F
-P 5750 2900
-F 0 "#FLG3" H 5750 2995 50  0001 C CNN
-F 1 "PWR_FLAG" H 5750 3080 50  0000 C CNN
-F 2 "" H 5750 2900 50  0000 C CNN
-F 3 "" H 5750 2900 50  0000 C CNN
-	1    5750 2900
+P 5750 2825
+F 0 "#FLG08" H 5750 2920 50  0001 C CNN
+F 1 "PWR_FLAG" H 5750 3005 50  0000 C CNN
+F 2 "" H 5750 2825 50  0000 C CNN
+F 3 "" H 5750 2825 50  0000 C CNN
+	1    5750 2825
 	1    0    0    -1
 $EndComp
@@
 F 0 "PD1" H 3650 2365 60  0000 C CNN
 F 1 "Hole" H 3650 2575 60  0000 C CNN
-F 2 "Mounting_Holes:MountingHole_3.2mm_M3" H 3650 2475 60  0001 C CNN
+F 2 "Custom:MountingHole_3.3mm_M3" H 3650 2475 60  0001 C CNN
 F 3 "" H 3650 2475 60  0000 C CNN
 	1    3650 2475
@@
 F 0 "PD2" H 3850 2365 60  0000 C CNN
 F 1 "Hole" H 3850 2575 60  0000 C CNN
-F 2 "Mounting_Holes:MountingHole_3.2mm_M3" H 3850 2475 60  0001 C CNN
+F 2 "Custom:MountingHole_3.3mm_M3" H 3850 2475 60  0001 C CNN
 F 3 "" H 3850 2475 60  0000 C CNN
 	1    3850 2475
@@
 F 0 "PD3" H 4050 2365 60  0000 C CNN
 F 1 "Hole" H 4050 2575 60  0000 C CNN
-F 2 "Mounting_Holes:MountingHole_3.2mm_M3" H 4050 2475 60  0001 C CNN
+F 2 "Custom:MountingHole_3.3mm_M3" H 4050 2475 60  0001 C CNN
 F 3 "" H 4050 2475 60  0000 C CNN
 	1    4050 2475
@@
 F 0 "PD4" H 4250 2365 60  0000 C CNN
 F 1 "Hole" H 4250 2575 60  0000 C CNN
-F 2 "Mounting_Holes:MountingHole_3.2mm_M3" H 4250 2475 60  0001 C CNN
+F 2 "Custom:MountingHole_3.3mm_M3" H 4250 2475 60  0001 C CNN
 F 3 "" H 4250 2475 60  0000 C CNN
 	1    4250 2475
 	1    0    0    -1
 $EndComp
+$Comp
+L CONN_01X02 P1
+U 1 1 57C2E687
+P 3750 2950
+F 0 "P1" H 3750 3100 50  0000 C CNN
+F 1 "V_IN" V 3850 2950 50  0000 C CNN
+F 2 "Custom:AKL_320-02" H 3750 2950 50  0001 C CNN
+F 3 "http://cdn-reichelt.de/documents/datenblatt/C100/AKL320%23RIA.pdf" H 3750 2950 50  0001 C CNN
+F 4 "Reichelt" H 3750 2950 60  0001 C CNN "Supply"
+F 5 "AKL 320-02" H 3750 2950 60  0001 C CNN "Part No."
+F 6 "http://www.reichelt.de/AKL-320-02/3/index.html?&ACTION=3&LA=446&ARTICLE=36672&artnr=AKL+320-02&SEARCH=AKL349" H 3750 2950 60  0001 C CNN "URL"
+F 7 "\"0,26\"" H 3750 2950 60  0001 C CNN "Price"
+F 8 "Buchse AKL 349-02" H 3750 2950 60  0001 C CNN "Spec"
+	1    3750 2950
+	-1   0    0    -1
+$EndComp
+Connection ~ 4000 2900
+Wire Wire Line
+	3950 3000 3950 3275
+Wire Wire Line
+	3950 3275 4200 3275
+Wire Wire Line
+	4000 3275 4000 3325
+Wire Wire Line
+	4200 3275 4200 3250
+Connection ~ 4000 3275
+Wire Wire Line
+	5750 2825 5750 2900
+Connection ~ 5750 2900
+Wire Wire Line
+	6025 3000 5750 3000
+Wire Wire Line
+	5750 3000 5750 3350
+$Comp
+L CONN_01X02 P2
+U 1 1 57C2EC72
+P 6225 2950
+F 0 "P2" H 6225 3100 50  0000 C CNN
+F 1 "V_OUT" V 6325 2950 50  0000 C CNN
+F 2 "Custom:AKL_320-02" H 6225 2950 50  0001 C CNN
+F 3 "http://cdn-reichelt.de/documents/datenblatt/C100/AKL320%23RIA.pdf" H 6225 2950 50  0001 C CNN
+F 4 "Reichelt" H 6225 2950 60  0001 C CNN "Supply"
+F 5 "AKL 320-02" H 6225 2950 60  0001 C CNN "Part No."
+F 6 "http://www.reichelt.de/AKL-320-02/3/index.html?&ACTION=3&LA=446&ARTICLE=36672&artnr=AKL+320-02&SEARCH=AKL349" H 6225 2950 60  0001 C CNN "URL"
+F 7 "\"0,26\"" H 6225 2950 60  0001 C CNN "Price"
+F 8 "Buchse AKL 349-02" H 6225 2950 60  0001 C CNN "Spec"
+	1    6225 2950
+	1    0    0    -1
+$EndComp

Commit message: - RC-Glieder im Schaltplan hinzugefügt - LED4 Hinzugefügt
Parts:
- removed P1: V_IN, Custom:AKL_320-02, symbol CONN_01X02
- removed P2: V_OUT, Custom:AKL_320-02, symbol CONN_01X02
- removed PD3, PD4: Hole, Custom:MountingHole_3.3mm_M3, symbol Hole
- added D1: LED, Custom:LED_0603_HandSoldering, symbol LED
- added P1: V_IN+, symbol CONN_01X01
- added P2: V_IN-, symbol CONN_01X01
- added P4, P5: V_OUT+, symbol CONN_01X01
- added R3: 3k6, symbol R_Small
- P3: renamed from uC_IN1; value SIL 3 -> uC_IN; Package 1x3 Header -> 1x3 Angled; Part No. (none) -> PS 25/3W BR; Price (none) -> \"0,42\"; Supply (none) -> Reichelt; URL (none) -> http://www.reichelt.de/PS-25-3W-BR/3/index.html?ACTION=3&LA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
Connections:
- wire segments 25 -> 27
Changed lines of the file:
@@
 $EndComp
 $Comp
-L CONN_01X03 uC_IN1
+L CONN_01X03 P3
 U 1 1 5783BAEB
 P 3750 3800
-F 0 "uC_IN1" H 3750 4000 50  0000 C CNN
-F 1 "SIL 3" V 3850 3800 50  0000 C CNN
+F 0 "P3" H 3750 4000 50  0000 C CNN
+F 1 "uC_IN" V 3850 3800 50  0000 C CNN
 F 2 "Pin_Headers:Pin_Header_Straight_1x03" H 3750 3800 50  0001 C CNN
-F 3 "" H 3750 3800 50  0000 C CNN
-F 4 "1x3 Header" H 3750 3800 60  0001 C CNN "Package"
+F 3 "http://cdn-reichelt.de/documents/datenblatt/C151/PS25_xxWBR.pdf" H 3750 3800 50  0001 C CNN
+F 4 "Reichelt" H 3750 3800 60  0001 C CNN "Supply"
+F 5 "PS 25/3W BR" H 3750 3800 60  0001 C CNN "Part No."
+F 6 "http://www.reichelt.de/PS-25-3W-BR/3/index.html?ACTION=3&LA=446&ARTICLE=14828&artnr=PS+25%2F3W+BR&SEARCH=PS+25" H 3750 3800 60  0001 C CNN "URL"
+F 7 "\"0,42\"" H 3750 3800 60  0001 C CNN "Price"
+F 8 "1x3 Angled" H 3750 3800 60  0001 C CNN "Package"
 	1    3750 3800
 	-1   0    0    -1
@@
 L GND #PWR05
 U 1 1 5783C5FB
-P 5750 3350
-F 0 "#PWR05" H 5750 3100 50  0001 C CNN
-F 1 "GND" H 5750 3200 50  0000 C CNN
-F 2 "" H 5750 3350 50  0000 C CNN
-F 3 "" H 5750 3350 50  0000 C CNN
-	1    5750 3350
+P 5925 3350
+F 0 "#PWR05" H 5925 3100 50  0001 C CNN
+F 1 "GND" H 5925 3200 50  0000 C CNN
+F 2 "" H 5925 3350 50  0000 C CNN
+F 3 "" H 5925 3350 50  0000 C CNN
+	1    5925 3350
 	1    0    0    -1
 $EndComp
@@
 	5550 2900 6025 2900
 Wire Wire Line
-	5750 3350 5750 3350
+	5925 3350 5925 3350
 $Comp
 L C_Small C1
@@
 	1    0    0    -1
 $EndComp
-$Comp
-L Hole PD3
-U 1 1 57ADE2E0
-P 4050 2475
-F 0 "PD3" H 4050 2365 60  0000 C CNN
-F 1 "Hole" H 4050 2575 60  0000 C CNN
-F 2 "Custom:MountingHole_3.3mm_M3" H 4050 2475 60  0001 C CNN
-F 3 "" H 4050 2475 60  0000 C CNN
-	1    4050 2475
-	1    0    0    -1
-$EndComp
-$Comp
-L Hole PD4
-U 1 1 57ADE320
-P 4250 2475
-F 0 "PD4" H 4250 2365 60  0000 C CNN
-F 1 "Hole" H 4250 2575 60  0000 C CNN
-F 2 "Custom:MountingHole_3.3mm_M3" H 4250 2475 60  0001 C CNN
-F 3 "" H 4250 2475 60  0000 C CNN
-	1    4250 2475
-	1    0    0    -1
-$EndComp
-$Comp
-L CONN_01X02 P1
-U 1 1 57C2E687
-P 3750 2950
-F 0 "P1" H 3750 3100 50  0000 C CNN
-F 1 "V_IN" V 3850 2950 50  0000 C CNN
-F 2 "Custom:AKL_320-02" H 3750 2950 50  0001 C CNN
-F 3 "http://cdn-reichelt.de/documents/datenblatt/C100/AKL320%23RIA.pdf" H 3750 2950 50  0001 C CNN
-F 4 "Reichelt" H 3750 2950 60  0001 C CNN "Supply"
-F 5 "AKL 320-02" H 3750 2950 60  0001 C CNN "Part No."
-F 6 "http://www.reichelt.de/AKL-320-02/3/index.html?&ACTION=3&LA=446&ARTICLE=36672&artnr=AKL+320-02&SEARCH=AKL349" H 3750 2950 60  0001 C CNN "URL"
-F 7 "\"0,26\"" H 3750 2950 60  0001 C CNN "Price"
-F 8 "Buchse AKL 349-02" H 3750 2950 60  0001 C CNN "Spec"
-	1    3750 2950
-	-1   0    0    -1
-$EndComp
 Connection ~ 4000 2900
-Wire Wire Line
-	3950 3000 3950 3275
 Wire Wire Line
 	3950 3275 4200 3275
@@
 Connection ~ 5750 2900
 Wire Wire Line
-	6025 3000 5750 3000
-Wire Wire Line
-	5750 3000 5750 3350
-$Comp
-L CONN_01X02 P2
-U 1 1 57C2EC72
-P 6225 2950
-F 0 "P2" H 6225 3100 50  0000 C CNN
-F 1 "V_OUT" V 6325 2950 50  0000 C CNN
-F 2 "Custom:AKL_320-02" H 6225 2950 50  0001 C CNN
-F 3 "http://cdn-reichelt.de/documents/datenblatt/C100/AKL320%23RIA.pdf" H 6225 2950 50  0001 C CNN
-F 4 "Reichelt" H 6225 2950 60  0001 C CNN "Supply"
-F 5 "AKL 320-02" H 6225 2950 60  0001 C CNN "Part No."
-F 6 "http://www.reichelt.de/AKL-320-02/3/index.html?&ACTION=3&LA=446&ARTICLE=36672&artnr=AKL+320-02&SEARCH=AKL349" H 6225 2950 60  0001 C CNN "URL"
-F 7 "\"0,26\"" H 6225 2950 60  0001 C CNN "Price"
-F 8 "Buchse AKL 349-02" H 6225 2950 60  0001 C CNN "Spec"
-	1    6225 2950
-	1    0    0    -1
-$EndComp
+	6025 3275 5925 3275
+Wire Wire Line
+	5925 3275 5925 3350
+$Comp
+L R_Small R3
+U 1 1 57C815D8
+P 5600 3175
+F 0 "R3" H 5630 3195 50  0000 L CNN
+F 1 "3k6" H 5630 3135 50  0000 L CNN
+F 2 "" H 5600 3175 50  0001 C CNN
+F 3 "" H 5600 3175 50  0000 C CNN
+	1    5600 3175
+	1    0    0    -1
+$EndComp
+$Comp
+L CONN_01X01 P1
+U 1 1 57C8181A
+P 3750 2900
+F 0 "P1" H 3750 3000 50  0000 C CNN
+F 1 "V_IN+" V 3850 2900 50  0000 C CNN
+F 2 "" H 3750 2900 50  0001 C CNN
+F 3 "" H 3750 2900 50  0000 C CNN
+	1    3750 2900
+	-1   0    0    1
+$EndComp
+$Comp
+L CONN_01X01 P2
+U 1 1 57C8188D
+P 3750 3275
+F 0 "P2" H 3750 3375 50  0000 C CNN
+F 1 "V_IN-" V 3850 3275 50  0000 C CNN
+F 2 "" H 3750 3275 50  0001 C CNN
+F 3 "" H 3750 3275 50  0000 C CNN
+	1    3750 3275
+	-1   0    0    1
+$EndComp
+$Comp
+L CONN_01X01 P4
+U 1 1 57C8199A
+P 6225 2900
+F 0 "P4" H 6225 3000 50  0000 C CNN
+F 1 "V_OUT+" V 6325 2900 50  0000 C CNN
+F 2 "" H 6225 2900 50  0001 C CNN
+F 3 "" H 6225 2900 50  0000 C CNN
+	1    6225 2900
+	1    0    0    -1
+$EndComp
+$Comp
+L CONN_01X01 P5
+U 1 1 57C81A43
+P 6225 3275
+F 0 "P5" H 6225 3375 50  0000 C CNN
+F 1 "V_OUT+" V 6325 3275 50  0000 C CNN
+F 2 "" H 6225 3275 50  0001 C CNN
+F 3 "" H 6225 3275 50  0000 C CNN
+	1    6225 3275
+	1    0    0    -1
+$EndComp
+$Comp
+L LED D1
+U 1 1 57C81BD8
+P 5600 3550
+F 0 "D1" H 5600 3650 50  0000 C CNN
+F 1 "LED" H 5600 3450 50  0000 C CNN
+F 2 "Custom:LED_0603_HandSoldering" H 5600 3550 50  0001 C CNN
+F 3 "" H 5600 3550 50  0000 C CNN
+	1    5600 3550
+	0    -1   -1   0
+$EndComp
+$Comp
+L GND #PWR09
+U 1 1 57C81C76
+P 5600 3825
+F 0 "#PWR09" H 5600 3575 50  0001 C CNN
+F 1 "GND" H 5600 3675 50  0000 C CNN
+F 2 "" H 5600 3825 50  0000 C CNN
+F 3 "" H 5600 3825 50  0000 C CNN
+	1    5600 3825
+	1    0    0    -1
+$EndComp
+Wire Wire Line
+	5600 3825 5600 3750
+Wire Wire Line
+	5600 3350 5600 3275
+Wire Wire Line
+	5600 3075 5600 2900
+Connection ~ 5600 2900
 $EndSCHEMATC

Commit message: - 5V_Servo Zusätzlich zur verfügung gestellt - Footprints für Pinleisten mit Verrigelung Hinzugefügt
Parts:
- P1, P2, P4, P5: footprint (none) -> Custom:Pad_SMD_3.5x10
- P3: footprint Pin_Headers:Pin_Header_Straight_1x03 -> Custom:PS25_3W_BR
- R3: footprint (none) -> Resistors_SMD:R_0603_HandSoldering
Changed lines of the file:
@@
 F 0 "P3" H 3750 4000 50  0000 C CNN
 F 1 "uC_IN" V 3850 3800 50  0000 C CNN
-F 2 "Pin_Headers:Pin_Header_Straight_1x03" H 3750 3800 50  0001 C CNN
+F 2 "Custom:PS25_3W_BR" H 3750 3800 50  0001 C CNN
 F 3 "http://cdn-reichelt.de/documents/datenblatt/C151/PS25_xxWBR.pdf" H 3750 3800 50  0001 C CNN
 F 4 "Reichelt" H 3750 3800 60  0001 C CNN "Supply"
@@
 F 0 "R3" H 5630 3195 50  0000 L CNN
 F 1 "3k6" H 5630 3135 50  0000 L CNN
-F 2 "" H 5600 3175 50  0001 C CNN
+F 2 "Resistors_SMD:R_0603_HandSoldering" H 5600 3175 50  0001 C CNN
 F 3 "" H 5600 3175 50  0000 C CNN
 	1    5600 3175
@@
 F 0 "P1" H 3750 3000 50  0000 C CNN
 F 1 "V_IN+" V 3850 2900 50  0000 C CNN
-F 2 "" H 3750 2900 50  0001 C CNN
+F 2 "Custom:Pad_SMD_3.5x10" H 3750 2900 50  0001 C CNN
 F 3 "" H 3750 2900 50  0000 C CNN
 	1    3750 2900
@@
 F 0 "P2" H 3750 3375 50  0000 C CNN
 F 1 "V_IN-" V 3850 3275 50  0000 C CNN
-F 2 "" H 3750 3275 50  0001 C CNN
+F 2 "Custom:Pad_SMD_3.5x10" H 3750 3275 50  0001 C CNN
 F 3 "" H 3750 3275 50  0000 C CNN
 	1    3750 3275
@@
 F 0 "P4" H 6225 3000 50  0000 C CNN
 F 1 "V_OUT+" V 6325 2900 50  0000 C CNN
-F 2 "" H 6225 2900 50  0001 C CNN
+F 2 "Custom:Pad_SMD_3.5x10" H 6225 2900 50  0001 C CNN
 F 3 "" H 6225 2900 50  0000 C CNN
 	1    6225 2900
@@
 F 0 "P5" H 6225 3375 50  0000 C CNN
 F 1 "V_OUT+" V 6325 3275 50  0000 C CNN
-F 2 "" H 6225 3275 50  0001 C CNN
+F 2 "Custom:Pad_SMD_3.5x10" H 6225 3275 50  0001 C CNN
 F 3 "" H 6225 3275 50  0000 C CNN
 	1    6225 3275
