File: kicad_SchalterFahrakku/Schalter_Fahrakku.kicad_pcb (KiCad board)
At the start: 2 copper layers, 55 x 25 mm, 31 parts, among them P1 V_IN+, P2 V_IN-, P3 uC_IN, P4 V_OUT+, P5 V_OUT-, Q1 IRLML6344, Q2 IPD90P03

Commit message: - Layout Schalterplatine
Parts:
- moved R3 22.8 mm to (121.7, 93.2), turned to 0 degrees
- moved D1 22.0 mm to (125.8, 93.2), turned to 180 degrees
- moved C1 1.58 mm to (128.2, 89.8)
- moved Q1 1.58 mm to (123.3, 89.8)
- moved R1 1.58 mm to (126.3, 89.8)
- moved R2 0.90 mm to (124.2, 85.0)
- moved C2 0.90 mm to (122.0, 85.0)
Routing:
- net /CTL_DRIVE: track 0.00 -> 32.6 mm
- net GND: track 0.00 -> 11.5 mm, vias 0 -> 2
- net Net-(C2-Pad2): track 0.00 -> 9.03 mm
- net Net-(P4-Pad1): track 0.00 -> 8.77 mm
- net Net-(C2-Pad1): track 0.00 -> 6.33 mm
- net Net-(D1-Pad2): track 0.00 -> 2.00 mm
- added copper zone on B.Cu, net GND
- added copper zone on F.Cu, net GND
- added copper zone on F.Cu, net Net-(C2-Pad1)
- added copper zone on F.Cu, net Net-(P4-Pad1)
Changed lines of the file:
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@@
   (general
     (links 19)
-    (no_connects 19)
-    (area 99.924999 69.924999 155.075001 95.075001)
+    (no_connects 2)
+    (area 99.924999 69.075 155.075001 115.300001)
     (thickness 1.6)
     (drawings 11)
-    (tracks 0)
+    (tracks 40)
     (zones 0)
     (modules 31)
@@
   )
   (module Capacitors_SMD:C_0603_HandSoldering (layer F.Cu)
-    (at 128.31 88.17 90)
+    (at 128.25 89.75 90)
     (descr "Capacitor SMD 0603, hand soldering")
     (tags "capacitor 0603")
@@
   )
   (module Capacitors_SMD:C_0603_HandSoldering (layer F.Cu)
-    (at 122 84.15 270)
+    (at 122 85.05 270)
     (descr "Capacitor SMD 0603, hand soldering")
     (tags "capacitor 0603")
@@
   )
   (module TO_SOT_Packages_SMD:SOT-23 (layer F.Cu)
-    (at 123.31 88.17 90)
+    (at 123.31 89.75 90)
     (descr "SOT-23, Standard")
     (tags SOT-23)
@@
   )
   (module Resistors_SMD:R_0603_HandSoldering (layer F.Cu)
-    (at 126.31 88.17 90)
+    (at 126.31 89.75 90)
     (descr "Resistor SMD 0603, hand soldering")
     (tags "resistor 0603")
@@
   )
   (module Resistors_SMD:R_0603_HandSoldering (layer F.Cu)
-    (at 124.2 84.1 270)
+    (at 124.2 85 270)
     (descr "Resistor SMD 0603, hand soldering")
     (tags "resistor 0603")
@@
   )
   (module Custom:LED_0603_HandSoldering (layer F.Cu)
-    (at 132.6 72.3 90)
+    (at 125.85 93.25 180)
     (descr "Resistor SMD 0603, hand soldering")
     (tags "resistor 0603")
     (attr smd)
-    (fp_text reference D1 (at -2.9 0 90) (layer F.SilkS)
-      (effects (font (size 1 1) (thickness 0.15)))
-    )
-    (fp_text value LED (at 0 1.9 90) (layer F.Fab)
+    (fp_text reference D1 (at -2.9 0 180) (layer F.SilkS)
+      (effects (font (size 1 1) (thickness 0.15)))
+    )
+    (fp_text value LED (at 0 1.9 180) (layer F.Fab)
       (effects (font (size 1 1) (thickness 0.15)))
     )
@@
     (fp_line (start 0.5 0.675) (end -0.5 0.675) (layer F.SilkS) (width 0.15))
     (fp_line (start -0.5 -0.675) (end 0.5 -0.675) (layer F.SilkS) (width 0.15))
-    (pad 1 smd rect (at -1.1 0 90) (size 1.2 0.9) (layers F.Cu F.Paste F.Mask)
+    (pad 1 smd rect (at -1.1 0 180) (size 1.2 0.9) (layers F.Cu F.Paste F.Mask)
       (net 2 GND))
-    (pad 2 smd rect (at 1.1 0 90) (size 1.2 0.9) (layers F.Cu F.Paste F.Mask)
+    (pad 2 smd rect (at 1.1 0 180) (size 1.2 0.9) (layers F.Cu F.Paste F.Mask)
       (net 5 "Net-(D1-Pad2)"))
     (model Resistors_SMD.3dshapes/R_0603_HandSoldering.wrl
@@
   )
   (module Resistors_SMD:R_0603_HandSoldering (layer F.Cu)
-    (at 130.7 72.3 90)
+    (at 121.65 93.25)
     (descr "Resistor SMD 0603, hand soldering")
     (tags "resistor 0603")
     (attr smd)
-    (fp_text reference R3 (at -3 0.1 90) (layer F.SilkS)
-      (effects (font (size 1 1) (thickness 0.15)))
-    )
-    (fp_text value 3k6 (at 0 1.9 90) (layer F.Fab)
+    (fp_text reference R3 (at -3 0.1) (layer F.SilkS)
+      (effects (font (size 1 1) (thickness 0.15)))
+    )
+    (fp_text value 3k6 (at 0 1.9) (layer F.Fab)
       (effects (font (size 1 1) (thickness 0.15)))
     )
@@
     (fp_line (start 0.5 0.675) (end -0.5 0.675) (layer F.SilkS) (width 0.15))
     (fp_line (start -0.5 -0.675) (end 0.5 -0.675) (layer F.SilkS) (width 0.15))
-    (pad 1 smd rect (at -1.1 0 90) (size 1.2 0.9) (layers F.Cu F.Paste F.Mask)
+    (pad 1 smd rect (at -1.1 0) (size 1.2 0.9) (layers F.Cu F.Paste F.Mask)
       (net 6 "Net-(P4-Pad1)"))
-    (pad 2 smd rect (at 1.1 0 90) (size 1.2 0.9) (layers F.Cu F.Paste F.Mask)
+    (pad 2 smd rect (at 1.1 0) (size 1.2 0.9) (layers F.Cu F.Paste F.Mask)
       (net 5 "Net-(D1-Pad2)"))
     (model Resistors_SMD.3dshapes/R_0603_HandSoldering.wrl
@@
   (gr_line (start 100 95) (end 155 95) (layer Edge.Cuts) (width 0.15))
   (gr_line (start 100 70) (end 100 95) (layer Edge.Cuts) (width 0.15))
+  (segment (start 117 87.006502) (end 117 80.814998) (width 0.25) (layer F.Cu) (net 1))
+  (segment (start 117 80.814998) (end 121.439999 76.374999) (width 0.25) (layer F.Cu) (net 1))
+  (segment (start 121.439999 76.374999) (end 126.374999 76.374999) (width 0.25) (layer F.Cu) (net 1))
+  (segment (start 126.374999 76.374999) (end 126.700001 76.700001) (width 0.25) (layer F.Cu) (net 1))
+  (segment (start 126.700001 76.700001) (end 127.5 77.5) (width 0.25) (layer F.Cu) (net 1))
+  (segment (start 124.31076 90.7) (end 121.876678 90.7) (width 0.25) (layer F.Cu) (net 1))
+  (segment (start 121.876678 90.7) (end 121.586729 90.410051) (width 0.25) (layer F.Cu) (net 1))
+  (segment (start 121.586729 90.410051) (end 121.586729 89.251727) (width 0.25) (layer F.Cu) (net 1))
+  (segment (start 121.586729 89.251727) (end 119.757503 87.422501) (width 0.25) (layer F.Cu) (net 1))
+  (segment (start 119.757503 87.422501) (end 117.415999 87.422501) (width 0.25) (layer F.Cu) (net 1))
+  (segment (start 117.415999 87.422501) (end 117 87.006502) (width 0.25) (layer F.Cu) (net 1))
+  (segment (start 126.31 90.85) (end 124.46076 90.85) (width 0.25) (layer F.Cu) (net 1))
+  (segment (start 124.46076 90.85) (end 124.31076 90.7) (width 0.25) (layer F.Cu) (net 1))
+  (segment (start 128.25 90.7) (end 126.46 90.7) (width 0.25) (layer F.Cu) (net 1))
+  (segment (start 126.46 90.7) (end 126.31 90.85) (width 0.25) (layer F.Cu) (net 1))
+  (segment (start 126.25 87.075736) (end 126.31 87.135736) (width 0.25) (layer F.Cu) (net 2))
+  (segment (start 126.31 87.135736) (end 126.31 88.65) (width 0.25) (layer F.Cu) (net 2))
+  (segment (start 127 86.75) (end 126.575736 86.75) (width 0.25) (layer F.Cu) (net 2))
+  (segment (start 126.575736 86.75) (end 126.25 87.075736) (width 0.25) (layer F.Cu) (net 2))
+  (segment (start 128.25 88.75) (end 127 87.5) (width 0.25) (layer B.Cu) (net 2))
+  (segment (start 127 87.5) (end 127 86.75) (width 0.25) (layer B.Cu) (net 2))
+  (via (at 127 86.75) (size 0.6) (drill 0.2) (layers F.Cu B.Cu) (net 2))
+  (segment (start 128.75 89.25) (end 128.25 88.75) (width 0.25) (layer B.Cu) (net 2))
+  (segment (start 128.75 93.25) (end 128.75 89.25) (width 0.25) (layer B.Cu) (net 2))
+  (segment (start 126.95 93.25) (end 128.75 93.25) (width 0.25) (layer F.Cu) (net 2))
+  (via (at 128.75 93.25) (size 0.6) (drill 0.2) (layers F.Cu B.Cu) (net 2))
+  (segment (start 122.5 77.5) (end 121.2 77.5) (width 0.5) (layer F.Cu) (net 3))
+  (segment (start 121.2 77.5) (end 119.2 79.5) (width 0.5) (layer F.Cu) (net 3))
+  (segment (start 119.2 79.5) (end 119.2 80.3745) (width 0.5) (layer F.Cu) (net 3))
+  (segment (start 119.2 80.3745) (end 119.2 81.7) (width 0.5) (layer F.Cu) (net 3))
+  (segment (start 122 86) (end 124.1 86) (width 0.5) (layer F.Cu) (net 4))
+  (segment (start 124.1 86) (end 124.2 86.1) (width 0.5) (layer F.Cu) (net 4))
+  (segment (start 119.2 86.272) (end 121.728 86.272) (width 0.5) (layer F.Cu) (net 4))
+  (segment (start 121.728 86.272) (end 122 86) (width 0.5) (layer F.Cu) (net 4))
+  (segment (start 122.31178 89.75) (end 122.31178 86.31178) (width 0.5) (layer F.Cu) (net 4))
+  (segment (start 122.31178 86.31178) (end 122 86) (width 0.5) (layer F.Cu) (net 4))
+  (segment (start 122.75 93.25) (end 124.75 93.25) (width 0.5) (layer F.Cu) (net 5))
+  (segment (start 120.55 93.25) (end 120.55 90.05) (width 0.5) (layer F.Cu) (net 6))
+  (segment (start 120.55 90.05) (end 120.5 90) (width 0.5) (layer F.Cu) (net 6))
+  (segment (start 120.5 90) (end 115 90) (width 0.5) (layer F.Cu) (net 6))
+  (zone (net 2) (net_name GND) (layer F.Cu) (hatch edge 0.508)
+    (connect_pads (clearance 0.508))
+    (min_thickness 0.254)
+    (fill yes (arc_segments 16) (thermal_gap 0.508) (thermal_bridge_width 0.508))
+    (polygon
+      (pts
+        (xy 100 95) (xy 100 70) (xy 155 70) (xy 155 95)
+      )
+    )
+  )
+  (zone (net 2) (net_name GND) (layer B.Cu) (hatch edge 0.508)
+    (connect_pads (clearance 0.508))
+    (min_thickness 0.254)
+    (fill yes (arc_segments 16) (thermal_gap 0.508) (thermal_bridge_width 0.508))
+    (polygon
+      (pts
+        (xy 100 95) (xy 100 70) (xy 155 70) (xy 155 95)
+      )
+    )
+  )
+  (zone (net 6) (net_name "Net-(P4-Pad1)") (layer F.Cu) (hatch edge 0.508)
+    (priority 1)
+    (connect_pads yes (clearance 0.508))
+    (min_thickness 0.254)
+    (fill yes (arc_segments 16) (thermal_gap 0.508) (thermal_bridge_width 0.508))
+    (polygon
+      (pts
+        (xy 116.5 88) (xy 120 88) (xy 120 92) (xy 109.5 92) (xy 109.5 80.5)
+        (xy 116.5 80.5) (xy 116.5 88)
+      )
+    )
+  )
+  (zone (net 3) (net_name "Net-(C2-Pad1)") (layer F.Cu) (hatch edge 0.508)
+    (priority 1)
+    (connect_pads yes (clearance 0.508))
+    (min_thickness 0.254)
+    (fill yes (arc_segments 16) (thermal_gap 0.508) (thermal_bridge_width 0.508) (smoothing chamfer))
+    (polygon
+      (pts
+        (xy 117.5 80.75) (xy 117.5 85) (xy 136 85) (xy 136 75) (xy 132 75)
+        (xy 132 80.75)
+      )
+    )
+  )
+  (zone (net 2) (net_name GND) (layer F.Cu) (hatch edge 0.508)
+    (priority 1)
+    (connect_pads yes (clearance 0.508))
+    (min_thickness 0.254)
+    (fill yes (arc_segments 16) (thermal_gap 0.508) (thermal_bridge_width 0.508) (smoothing chamfer))
+    (polygon
+      (pts
+        (xy 141 74) (xy 141 85.75) (xy 146 85.75) (xy 146 74)
+      )
+    )
+  )
+  (zone (net 2) (net_name GND) (layer F.Cu) (hatch edge 0.508)
+    (priority 1)
+    (connect_pads yes (clearance 0.508))
+    (min_thickness 0.254)
+    (fill yes (arc_segments 16) (thermal_gap 0.508) (thermal_bridge_width 0.508) (smoothing chamfer))
+    (polygon
+      (pts
+        (xy 109.044516 77.5) (xy 120.794516 77.5) (xy 120.794516 72.5) (xy 109.044516 72.5)
+      )
+    )
+  )
 )
